File: Untitled/MCU.kicad_sch (KiCad schematic)
At the start: 31 parts, among them J1 Conn_02x07_Top_Bottom, U1 STM32F070CBT6TR, Y1 ABM8G-12.000MHZ-18-D2Y-T

Commit message: revised verison
Parts:
- removed C1: 1uF, Capacitor_SMD:C_0805_2012Metric_Pad1.18x1.45mm_HandSolder, symbol Device:C_Small
- removed C12, C15, C18, C21, C24: 0.1uF, Capacitor_SMD:C_0805_2012Metric_Pad1.18x1.45mm_HandSolder, symbol Device:C_Small
- removed C3: 10nF, Capacitor_SMD:C_0805_2012Metric_Pad1.18x1.45mm_HandSolder, symbol Device:C_Small
- removed C37, C38: 6pF, Capacitor_SMD:C_0603_1608Metric_Pad1.08x0.95mm_HandSolder, symbol Device:C_Small
- removed C9: 4.7uF, Capacitor_SMD:C_0805_2012Metric_Pad1.18x1.45mm_HandSolder, symbol Device:C_Small
- removed JP1: Jumper_2_Bridged, Connector_PinHeader_2.54mm:PinHeader_1x02_P2.54mm_Vertical, symbol Jumper:Jumper_2_Bridged
- removed MCLK1: 4952, USB-c:KEYSTONE_4952, symbol 4925:4952
- removed U1: STM32F070CBT6TR, USB-c:LQFP48-7x7mm, symbol Stm32f:STM32F070CBT6TR
- removed Y1: ABM8G-12.000MHZ-18-D2Y-T, USB-c:CRYSTAL_ABM8G_ABR, symbol Clock:ABM8G-12.000MHZ-18-D2Y-T
- added AGND1, GND1, MISO1, MOSI1, SCLK1: 4952, USB-c:KEYSTONE_4952, symbol 4925:4952
- added C1, C10, C2, C3, C4, C5: 1uF, Capacitor_SMD:C_0805_2012Metric_Pad1.18x1.45mm_HandSolder, symbol Device:C
- added D10, D11, D9: GREEN LED, LED_SMD:LED_1206_3216Metric_Pad1.42x1.75mm_HandSolder, symbol Device:LED
- added D8: RED LED, LED_SMD:LED_1206_3216Metric_Pad1.42x1.75mm_HandSolder, symbol Device:LED
- added R10, R11, R12, R9: 220R, Resistor_SMD:R_0805_2012Metric_Pad1.20x1.40mm_HandSolder, symbol Device:R_US
- added S5: GF-123-0054, USB-c:SW_GF-123-0054, symbol GF-123-0054:GF-123-0054
- added U1: STM32H523VET6, USB-c:LQFP-100, symbol stm32h:STM32H523VET6
- J1: value Conn_02x07_Top_Bottom -> Debugging Connector
Connections:
- net +3.3VD: now also C1.2, C10.2, C2.1, C3.1, C4.1, C5.1, S5.2, U1.100 (VDD), U1.11 (VDD), U1.22 (VDDA), U1.28 (VDD), U1.50 (VDD), U1.73 (VDDUSB), U1.75 (VDD)
- net CUR_SEN: now also U1.36 (PB1)
- net GND: now also AGND1.TP, C1.1, C10.1, C2.2, C3.2, C4.2, C5.2, GND1.TP, U1.10 (VSS), U1.19 (VSSA), U1.27 (VSS), U1.49 (VSS), U1.74 (VSS), U1.99 (VSS)
- net MCLCK_IN: now also U1.12 (PH0-OSC_IN)
- net MCLCK_OUT: now also U1.13 (PH1-OSC_OUT)
- net MCLR: now also U1.14 (NRST)
- net PGC: now also U1.72 (PA13)
- net PGD: now also U1.76 (PA14)
- net UART_RX: now also U1.54 (PB15)
- net UART_TX: now also U1.53 (PB14)
- net USB_DM: now also U1.70 (PA11)
- net USB_DP: now also U1.71 (PA12)
- net ADC_LED: now reaches D1.2 (A), D2.2 (A), D3.2 (A), D4.2 (A), D5.2 (A), D6.2 (A)
- net ADC_LED: now also D10.2 (A), D11.2 (A), D8.2 (A), D9.2 (A), S5.1
- net at R5.2: now also U1.26 (PA3)
- net at R6.2: now also U1.25 (PA2)
- net at R8.2: now also U1.23 (PA0)
- net at R7.2: now also U1.24 (PA1)
- net at R4.2: now also U1.29 (PA4)
- net at R3.2: now also U1.68 (PA9)
- new net: D9.1 (K), R10.1
- new net: R10.2, U1.18 (PC3)
- new net: D11.1 (K), R12.1
- new net: D8.1 (K), R9.1
- new net: R9.2, U1.4 (PE5)
- new net: R11.2, U1.16 (PC1)
- new net: R12.2, U1.66 (PC9)
- new net: D10.1 (K), R11.1
- new net CS_ADC: U1.46 (PE15)
- new net HARD_ADC_COMP: U1.17 (PC2)
- new net HARD_BYPASS_MOSFET: U1.5 (PE6)
- new net HARD_LAS_ENB: U1.15 (PC0)
- new net IRQ: U1.47 (PB10)
- new net MISO: MISO1.TP, U1.44 (PE13)
- new net MOSI: MOSI1.TP, U1.45 (PE14)
- new net PIN_BYPASS_MOSFET: U1.41 (PE10)
- new net PIN_LAS_ENB: U1.39 (PE8)
- new net PIN_SWAP_ADC: U1.40 (PE9)
- new net REF_CLK: U1.67 (PA8)
- new net SCLK: SCLK1.TP, U1.43 (PE12)
- no-connect marks 33 -> 63
Other:
- added sheet Physical Switches & External Clock (Switch/Clock.kicad_sch)
- note removed: "C5=C6=2*(C_L - C_S) C_L = 8 C_S = 5 C5=C6=6 Source: https://microchip.my.site.com/s/article/Calculating-crystal-load-capacitor"
- moved on the sheet: D1, D2, D3, D4, D5, D6, J1, R3, R4, R5, R6, R7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
