File: Untitled/Amplifer.kicad_sch (KiCad schematic)
At the start: 6 parts, among them U7 MCP6L01x-xLT, U8 AP331AWG-7

Commit message: revised verison
Parts:
- added C6, C8: 0.1uF, Capacitor_SMD:C_0805_2012Metric_Pad1.18x1.45mm_HandSolder, symbol Device:C
- added C7, C9: 10uF, Capacitor_SMD:C_0805_2012Metric_Pad1.18x1.45mm_HandSolder, symbol Device:C
- added U10: ADG1419BRMZ, RM_8_ADI, symbol ADG1419BRMZ:ADG1419BRMZ
- added U11: MCP3462-E/ST, USB-c:TSSOP20_ST_MCH_MIS, symbol MCP3462:MCP3462-E_ST
Connections:
- net +3.3VD: now also C8.1, C9.1, U11.20 (DVDD); no longer C39.1, U7.5 (V+)
- net +5V: now also C39.1, U7.5 (V+), U10.4 (VDD)
- net GND: now also C6.2, C7.2, C8.2, C9.2, U10.3 (GND), U10.7 (VSS), U11.19 (DGND), U11.2 (AGND), U11.3 (REFIN-)
- net at C36.2, R2.2, U7.1: now also U10.1 (D); no longer U8.3 (IN+)
- new net: U10.2 (SA), U11.5 (CH0)
- new net: U10.8 (SB), U8.3 (IN+)
- new net +3.3VA: C6.1, C7.1, U11.1 (AVDD), U11.4 (REFIN+)
- new net CLCK_REF: U11.18 (MCLKIN)
- new net CS_ADC: U11.13 (*CS)
- new net IRQ: U11.17 (*IRQ/MDAT)
- new net MISO: U11.16 (SDO)
- new net MOSI: U11.15 (SDI)
- new net PIN_SWAP_ADC: U10.6 (IN)
- new net SCLK: U11.14 (SCK)
- no-connect marks 0 -> 1
Other:
- note added: "ANALOG SPEFICS SWITCH"
- moved on the sheet: U8

Commit message: schematic updates
Other:
- note added: "Waiting on email reply to complete the numbers for these"
Changed lines of the file:
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@@
+		)
+	)
+	(text "Waiting on email reply to complete the numbers for these"
+		(exclude_from_sim no)
+		(at 76.962 131.064 0)
+		(effects
+			(font
+				(size 1.27 1.27)
+			)
 		)
 	)
