File: Untitled/Laser.kicad_sch (KiCad schematic)
At the start: 4 parts, among them J3 Screw_Terminal_01x02, U6 AL5809-20QP1-7

Commit message: revised verison
Parts:
- added MOSFET2: 2N7002, USB-c:SOT-23TO-236_318-08_ONS, symbol 2N7002:2N7002
- added U9: SN74LVC1G332DCKR, DCK0006A_N, symbol SN74LVC1G332DCKR:SN74LVC1G332DCKR
Connections:
- net +3.3VA: now also MOSFET2.3 (D); no longer U6.1 (IN)
- net GND: now also U9.2 (GND)
- net UART_TX: now also U9.1 (A); no longer MOSFET1.1 (G)
- new net: MOSFET1.1 (G), U9.4 (Y)
- new net: MOSFET2.2 (S), U6.1 (IN)
- new net +5V: U9.5 (VCC)
- new net LAS_ENB: MOSFET2.1 (G)
- new net PIN_BYPASS_MOSFET: U9.6 (C)
- no-connect marks 0 -> 1
Other:
- note added: "OR GATE UART SIGNALS CHANGES RAPIDLY (ANNOYING TO PROGRAME IF STABLE SIGNAL IS WANTED) BYPASS_MOSFET WILL BE A STABLE ON/OFF STATE"
- note added: "Screw terminal for laser Laser datasheet: https://mm.digikey.com/Volume0/opasdata/d220001/medias/docus/1130/1054_Web.pdf"
- note added: "Want UART TX signals to create laser pulses UART 0 signals expect no laser pulse UART 1 signals expect strong (max 25mA) laser pulse Expect signals to change fast"
- note removed: "Screw terminal for laser Laser datasheet:"
- note removed: "Want UART TX signals to create laser pulses UART 0 signals expect no laser pulse UART 1 signals expect strong (max 150mA) laser pulse Expect signals to change fast"

Commit message: fixed board
Parts:
- removed LAS1: 4952, USB-c:KEYSTONE_4952, symbol 4925:4952
Changed lines of the file:
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@@
 		)
-	)
-	(junction
-		(at 99.06 97.79)
-		(diameter 0)
-		(color 0 0 0 0)
 	)
 	(no_connect
@@
 	(wire
 		(pts
-			(xy 86.36 97.79) (xy 99.06 97.79)
-		)
-		(stroke
-			(width 0)
-			(type default)
-		)
-	)
-	(wire
-		(pts
 			(xy 59.69 107.95) (xy 59.69 114.3)
 		)
@@
 	(wire
 		(pts
-			(xy 99.06 97.79) (xy 121.92 97.79)
+			(xy 86.36 97.79) (xy 121.92 97.79)
 		)
 		(stroke
@@
 					(unit 1)
 				)
-			)
-		)
-	)
-	(symbol
-		(lib_id "4925:4952")
-		(at 99.06 92.71 90)
-		(unit 1)
-		(exclude_from_sim no)
-		(in_bom yes)
-		(on_board yes)
-		(dnp no)
-		(fields_autoplaced yes)
-		(property "Reference" "LAS1"
-			(at 101.6 91.4399 90)
-			(effects
-				(font
-					(size 1.27 1.27)
-				)
-				(justify right)
-			)
-		)
-		(property "Value" "4952"
-			(at 101.6 93.9799 90)
-			(effects
-				(font
-					(size 1.27 1.27)
-				)
-				(justify right)
-			)
-		)
-		(property "Footprint" "USB-c:KEYSTONE_4952"
-			(at 99.06 92.71 0)
-			(effects
-				(font
-					(size 1.27 1.27)
-				)
-				(justify bottom)
-				(hide yes)
-			)
-		)
-		(property "Datasheet" ""
-			(at 99.06 92.71 0)
-			(effects
-				(font
-					(size 1.27 1.27)
-				)
-				(hide yes)
-			)
-		)
-		(property "Description" ""
-			(at 99.06 92.71 0)
-			(effects
-				(font
-					(size 1.27 1.27)
-				)
-				(hide yes)
-			)
-		)
-		(property "PARTREV" "A"
-			(at 99.06 92.71 0)
-			(effects
-				(font
-					(size 1.27 1.27)
-				)
-				(justify bottom)
-				(hide yes)
-			)
-		)
-		(property "STANDARD" "Manufacturer Recommendations"
-			(at 99.06 92.71 0)
-			(effects
-				(font
-					(size 1.27 1.27)
-				)
-				(justify bottom)
-				(hide yes)
-			)
-		)
-		(property "SNAPEDA_PN" "4952"
-			(at 99.06 92.71 0)
-			(effects
-				(font
-					(size 1.27 1.27)
-				)
-				(justify bottom)
-				(hide yes)
-			)
-		)
-		(property "MAXIMUM_PACKAGE_HEIGHT" "6.3mm"
-			(at 99.06 92.71 0)
-			(effects
-				(font
-					(size 1.27 1.27)
-				)
-				(justify bottom)
-				(hide yes)
-			)
-		)
-		(property "MANUFACTURER" "Keystone"
-			(at 99.06 92.71 0)
-			(effects
-				(font
-					(size 1.27 1.27)
-				)
-				(justify bottom)
-				(hide yes)
-			)
-		)
-		(pin "TP"
-		)
-		(instances
-			(project "Untitled"
-				(path "/ad09c7d2-efab-4012-a18d-674ee0550e5f/e170c99a-257e-4de8-a63c-9467f11c5f52"
-					(reference "LAS1")
-					(unit 1)
-				)
