File: Untitled/Untitled.kicad_sch (KiCad schematic)
At the start: 0 parts

Commit message: revised verison
Other:
- sheet Analog Amplifer ports: added CLCK_REF, CS_ADC, IRQ, MISO, MOSI, PIN_SWAP_ADC, SCLK; removed none
- sheet Laser ports: added LAS_ENB, PIN_BYPASS_MOSFET; removed none
- sheet MCU ports: added CS_ADC, IRQ, MISO, MOSI, PIN_BYPASS_MOSFET, PIN_LAS_ENB, PIN_SWAP_ADC, REF_CLK, SCLK; removed none

Commit message: fixed board
Other:
- sheet Power ports: added DN, DP; removed DATA1, DATA2
Changed lines of the file:
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@@
+	(wire
+		(pts
+			(xy 58.42 97.79) (xy 58.42 125.73)
+		)
+		(stroke
+			(width 0)
+			(type default)
+		)
+	)
 	(wire
 		(pts
@@
 	(wire
 		(pts
+			(xy 55.88 97.79) (xy 55.88 125.73)
+		)
+		(stroke
+			(width 0)
+			(type default)
+		)
+	)
+	(wire
+		(pts
 			(xy 113.03 143.51) (xy 116.84 143.51)
 		)
@@
 	(wire
 		(pts
-			(xy 55.88 97.79) (xy 55.88 125.73)
-		)
-		(stroke
-			(width 0)
-			(type default)
-		)
-	)
-	(wire
-		(pts
 			(xy 43.18 97.79) (xy 43.18 125.73)
 		)
@@
 		(pts
 			(xy 66.04 97.79) (xy 66.04 102.87)
-		)
-		(stroke
-			(width 0)
-			(type default)
-		)
-	)
-	(wire
-		(pts
-			(xy 58.42 97.79) (xy 58.42 125.73)
 		)
 		(stroke
@@
 			)
 		)
-		(pin "DATA1" bidirectional
+		(pin "DN" bidirectional
+			(at 58.42 125.73 90)
+			(effects
+				(font
+					(size 1.27 1.27)
+				)
+				(justify right)
+			)
+		)
+		(pin "DP" bidirectional
 			(at 55.88 125.73 90)
 			(effects
 				(font
-					(size 1.27 1.27)
-				)
-				(justify right)
-			)
-		)
-		(pin "DATA2" bidirectional
-			(at 58.42 125.73 90)
-			(effects
-				(font
