File: Untitled/Switch/Clock.kicad_sch (KiCad schematic)
At the start: 6 parts, among them Y1 ABM8G-12.000MHZ-18-D2Y-T

Commit message: schematic updates
Other:
- note added: "hardware switches"
Changed lines of the file:
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@@
 	(generator_version "9.0")
 	(paper "A4")
+	(rectangle
+		(start 34.29 43.18)
+		(end 152.4 119.38)
+		(stroke
+			(width 0)
+			(type default)
+		)
+		(fill
+			(type none)
+		)
+	)
 	(text "C5=C6=2*(C_L - C_S)\n\nC_L = 8 \nC_S = 5\n\nC5=C6=6\n\nSource: https://microchip.my.site.com/s/article/Calculating-crystal-load-capacitor"
 		(exclude_from_sim no)
@@
 			)
 		)
+	)
+	(text "hardware switches"
+		(exclude_from_sim no)
+		(at 108.458 55.118 0)
+		(effects
+			(font
+				(size 2 2)
+			)
+		)
